Commit message: feat(sim): add in urdf file and convert urdf into xml with some tweaks

File: sim/description/urdf/TonyPi.urdf (robot description, URDF)
Before this commit: robot tonypi, 17 links, 16 joints
Links:
- added link L_hand, mass 0.05; collision box size=0.05 0.03 0.01; visual box size=0.05 0.03 0.01
- added link R_hand, mass 0.05; collision box size=0.05 0.03 0.01; visual box size=0.05 0.03 0.01
- link L_hip: mass None -> 0.001
- link L_shoulder: mass None -> 0.001
- link R_hip: mass None -> 0.001
- link R_shoulder: mass None -> 0.001
- link neck: mass None -> 0.001
Joints:
- added joint L_wrist: type revolute, parent L_forearm, child L_hand, origin xyz=0 0.06 0 rpy=0 0 0, axis 0 1 0, limit lower=-2.0 upper=2.0 effort=4 velocity=6
- added joint R_wrist: type revolute, parent R_forearm, child R_hand, origin xyz=0 -0.06 0 rpy=0 0 0, axis 0 1 0, limit lower=-2.0 upper=2.0 effort=4 velocity=6
